File: RC3.sch (KiCad schematic (older format))
At the start: 47 parts, among them P1 CONN_2, P2 CONN_3, P3 CONN_3X2, P4 CONN_2, Q1 MOSFET_N, Q10 MOSFET_N, Q11 MOSFET_N, Q12 MOSFET_N, Q13 MOSFET_N, Q14 MOSFET_N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

Commit message: fucked up merging new-lib
Parts:
- added C11: 1u, ~, symbol C
- added C12: 47n, ~, symbol C
- added D1, D2, D3: DIODE, ~, symbol DIODE
- added R15, R16, R17, R18, R19, R20: 10K, ~, symbol R
Connections:
- wire segments 239 -> 269
