File: RC3.kicad_pcb (KiCad board)
At the start: 2 copper layers, 84.8 x 91.4 mm, 47 parts, among them P1 CONN_2, P2 CONN_3, P3 CONN_3X2, P4 CONN_2, Q1 MOSFET_N, Q10 MOSFET_N, Q11 MOSFET_N, Q12 MOSFET_N, Q13 MOSFET_N, Q14 MOSFET_N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

Commit message: fucked up merging new-lib
Parts:
- added 1PIN: P***, 1pin, F.Cu at (146.7, 222.9)
- added 1PIN: P***, 1pin, F.Cu at (221.6, 222.2)
- added 1PIN: P***, 1pin, F.Cu at (222.2, 139.7)
- added ?: P***, 1PIN_SMD, F.Cu at (215.4, 162.7)
- added C11: 1u, SM1210, F.Cu at (175.3, 151.4)
- added C12: 47n, SM1206, F.Cu at (190.5, 151.4)
- added D1: DIODE, DO-214AC(SMA), F.Cu at (175.3, 168.9)
- added D2: DIODE, DO-214AC(SMA), F.Cu at (189.9, 168.9)
- added D3: DIODE, DO-214AC(SMA), F.Cu at (203.8, 168.9)
- added R15: 10K, SM1206, F.Cu at (203.5, 140.5)
- added R16: 10K, SM1206, F.Cu at (203.5, 144.5)
- added R17: 10K, SM1206, F.Cu at (203.5, 148.3)
- added R18: 10K, SM1206, F.Cu at (196.6, 144.5)
- added R19: 10K, SM1206, F.Cu at (196.6, 140.5)
- added R20: 10K, SM1206, F.Cu at (196.6, 148.3)
- moved P4 12.7 mm to (184.2, 143.5)
- moved R4 7.65 mm to (175.3, 222.9)
- moved R5 7.65 mm to (175.3, 219.1)
- moved R6 7.65 mm to (190.5, 222.9)
- moved R7 7.65 mm to (190.5, 219.1)
- moved R8 7.65 mm to (204.5, 222.9)
- moved R9 7.65 mm to (204.5, 219.1)
- moved R3 6.73 mm to (203.5, 154.9)
- moved R12 6.65 mm to (203.5, 151.6)
- moved Q6 4.33 mm to (197.1, 218.9), turned to 90 degrees
- moved Q2 4.32 mm to (167.6, 218.9), turned to 90 degrees
- moved Q4 4.32 mm to (182.9, 218.9), turned to 90 degrees
- moved Q12 3.31 mm to (197.1, 207.8), turned to 90 degrees
- moved Q10 3.30 mm to (182.9, 207.8), turned to 90 degrees
- moved Q8 3.30 mm to (167.6, 207.8), turned to 90 degrees
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Routing:
- net OUT_C: track 169.2 -> 223.6 mm, vias 0 -> 3
- net OUT_A: track 170.1 -> 223.2 mm, vias 0 -> 2
- net OUT_B: track 164.2 -> 210.8 mm, vias 0 -> 3
- net +5V: track 78.0 -> 122.5 mm, vias 2 -> 3
- net GND: track 323.0 -> 359.8 mm, vias 4 -> 3
- net N-000009: track 32.1 -> 59.6 mm
- net N-0000017: track 96.8 -> 76.3 mm
- net PWM: track 15.4 -> 35.1 mm, vias 0 -> 1
- net N-000001: track 29.6 -> 48.8 mm
- net ESTOPn: track 17.2 -> 36.4 mm, vias 0 -> 1
- net N-0000014: track 32.1 -> 51.1 mm, vias 0 -> 1
- net N-000008: track 29.6 -> 48.5 mm
- net N-000004: track 32.1 -> 50.3 mm, vias 0 -> 1
- net DIREC: track 21.6 -> 39.7 mm, vias 1 -> 2
- net N-0000015: track 29.6 -> 47.2 mm
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- removed copper zone on F.Cu, net GND
